File: Hardware/Motherboard.kicad_pcb (KiCad board)
At the start: 4 copper layers, 67.3 x 78.7 mm, 45 parts, among them J1 Pin_Header_02x08, J2 Pin_Header_02x08, J3 Pin_Header_02x08, J4 USB_B_Mini, J5 JTAG, SW1 SW_SPDT, U1 PIC18F26K22-I-SO, U2 FT240XS, U3 TXB0104D, U4 TXB0104D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

Commit message: [Hardware] Finished PCB routing. Switched two schematic signals to help routing.
Parts:
- moved C24 52.6 mm to (143.3, 120.7)
- moved C9 48.4 mm to (112.0, 99.1)
- moved C11 48.2 mm to (113.0, 94.9)
- moved C22 48.2 mm to (143.3, 123.2)
- moved C14 47.8 mm to (120.7, 108.0), turned to 270 degrees
- moved C13 47.2 mm to (112.0, 101.6)
- moved C10 47.2 mm to (115.6, 94.2)
- moved C15 46.9 mm to (114.9, 116.8)
- moved C16 46.9 mm to (121.0, 116.8)
- moved C6 46.9 mm to (134.0, 83.6)
- moved C7 46.9 mm to (137.6, 81.9)
- moved D1 46.9 mm to (134.0, 58.4)
- moved R3 46.9 mm to (113.7, 109.4)
- moved C1 46.9 mm to (112.4, 70.5)
- moved C17 46.9 mm to (150.2, 80.0)
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Connections:
- U1 pad 23: /FTDI_RD -> /FTDI_WR
- U1 pad 24: /FTDI_WR -> /FTDI_RD
Routing:
- net +5V: track 46.7 -> 232.4 mm, vias 0 -> 2
- net Net-(U1-Pad2): track 0.00 -> 41.6 mm, vias 0 -> 2
- net Net-(U1-Pad6): track 0.00 -> 38.1 mm, vias 0 -> 2
- net /TRANSLATOR_VCC: track 6.65 -> 44.5 mm, vias 0 -> 3
- net Net-(U1-Pad3): track 0.00 -> 36.8 mm, vias 0 -> 2
- net /FTDI_RD: track 0.00 -> 36.5 mm, vias 0 -> 2
- net Net-(U1-Pad5): track 0.00 -> 36.2 mm, vias 0 -> 2
- net Net-(U1-Pad4): track 0.00 -> 35.4 mm, vias 0 -> 2
- net Net-(U1-Pad7): track 0.00 -> 35.1 mm, vias 0 -> 2
- net Net-(U1-Pad10): track 0.00 -> 33.1 mm, vias 0 -> 2
- net /FTDI_WR: track 0.00 -> 32.9 mm, vias 0 -> 2
- net /FTDI_SIWU: track 0.00 -> 32.8 mm, vias 0 -> 2
- net Net-(U1-Pad9): track 0.00 -> 32.8 mm, vias 0 -> 2
- net /FTDI_TXE: track 0.00 -> 32.0 mm, vias 0 -> 2
- net /FTDI_RXF: track 0.00 -> 29.0 mm, vias 0 -> 2
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- added copper zone on B.Cu, net GND
- added copper zone on F.Cu, net GND
- added copper zone on In2.Cu, net GND
Other:
- board text added: "15/04/2020"
