File: Hardware/Logic_Signal_Generator.kicad_sch (KiCad schematic)
At the start: 18 parts, among them J1 JTAG, J3 USB_B, U1 PIC18F25K50-xSO

Commit message: [Hardware] Moved the LEDs description text to the Description field into the schematic."
Parts:
- D1: Value2 POWER -> (none)
- D2: Value2 USB_ACTIVITY -> (none)
Changed lines of the file:
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@@
 			)
 		)
-		(property "Description" ""
-			(at 77.47 160.02 0)
-			(effects
-				(font
-					(size 1.27 1.27)
-				)
-				(hide yes)
-			)
-		)
-		(property "Value2" "USB_ACTIVITY"
+		(property "Description" "USB_ACTIVITY"
 			(at 81.28 164.1474 90)
 			(effects
@@
 			)
 		)
-		(property "Description" ""
-			(at 48.26 160.02 0)
-			(effects
-				(font
-					(size 1.27 1.27)
-				)
-				(hide yes)
-			)
-		)
-		(property "Value2" "POWER"
+		(property "Description" "POWER"
 			(at 52.07 164.1474 90)
 			(effects
